File: quad_sipm_S133606025PE_5_2/_autosave-quad_sipm.sch (KiCad schematic (older format))
At the start: 18 parts, among them J1 8-102202-4, J2 8-102202-4, J3 8-102202-4, J4 8-102202-4

Commit message: added Rev 8.1: attenuator switch
Parts:
- removed J?: 8-102202-4, Connector_PinHeader_2.54mm:PinHeader_1x03_P2.54mm_Vertical, symbol Connector:Conn_01x03_Female
- D1, D2, D3, D4: symbol quad_sipm-rescue:D_Sipm_Quad-quad_sipm_symbols -> quad_sipm_symbols:D_Sipm_Quad
Changed lines of the file:
@@
 EESchema Schematic File Version 5
-EELAYER 36 0
+EELAYER 43 0
 EELAYER END
 $Descr A4 11693 8268
@@
 $EndComp
 $Comp
-L Connector:Conn_01x03_Female J?
-U 1 1 00000000
-P 5500 1950
-F 0 "J?" H 5650 2050 50  0000 C CNN
-F 1 "8-102202-4" H 5600 2200 50  0000 C CNN
-F 2 "Connector_PinHeader_2.54mm:PinHeader_1x03_P2.54mm_Vertical" H 5500 1950 50  0001 C CNN
-F 3 "~" H 5500 1950 50  0001 C CNN
-F 4 "A32559-ND" H 5450 2300 50  0000 C CNN "DigiKey"
-	1    5500 1950
-	-1   0    0    -1
-$EndComp
-$Comp
-L quad_sipm-rescue:D_Sipm_Quad-quad_sipm_symbols D1
+L quad_sipm_symbols:D_Sipm_Quad D1
 U 1 1 629A6BAF
 P 2500 1300
@@
 $EndComp
 $Comp
-L quad_sipm-rescue:D_Sipm_Quad-quad_sipm_symbols D2
+L quad_sipm_symbols:D_Sipm_Quad D2
 U 1 1 629A8647
 P 2500 2050
@@
 $EndComp
 $Comp
-L quad_sipm-rescue:D_Sipm_Quad-quad_sipm_symbols D3
+L quad_sipm_symbols:D_Sipm_Quad D3
 U 1 1 629A37BE
 P 4250 1300
@@
 $EndComp
 $Comp
-L quad_sipm-rescue:D_Sipm_Quad-quad_sipm_symbols D4
+L quad_sipm_symbols:D_Sipm_Quad D4
 U 1 1 629A5528
 P 4250 2050
