File: quad_sipm_S133606025PE_5_2/quad_sipm.kicad_sch (KiCad schematic)
At the start: 21 parts, among them J1 8-102202-4, J2 8-102202-4, J3 8-102202-4, J4 8-102202-4

Commit message: added Rev 8.1: attenuator switch
Parts:
- removed C1, C2, C3, C4: 10nF 100V, Capacitor_SMD:C_1206_3216Metric_Pad1.33x1.80mm_HandSolder, symbol Device:C_Small
- removed D1, D2, D3, D4: 1N914, Diode_SMD:S13360-6025PE, symbol Diode:1N914
- removed J1, J2, J3, J4: 8-102202-4, Connector_PinHeader_2.54mm:PinHeader_1x03_P2.54mm_Vertical, symbol Connector:Conn_01x03_Female
- removed R1, R2, R3, R4: R, Resistor_SMD:1206_VIS-L, symbol Device:R
Other:
- note removed: "Note: connector P/N is for right angle version"
